Commit message: Update centuar1.urdf

File: assets/urdf/centuar1.urdf (robot description, URDF)
Before this commit: robot 323Assembase_limit3, 39 links, 38 joints
Links:
- link wheel_right_link_1: geometry collision mesh filename=../meshes/wheel__link_1.stl scale=0.001 0.001 0.001; visual mesh filename=../meshes/wheel_left_link_1.stl scale=0.001 0.001 0.001
Joints:
- joint l_el: limit lower=-1.9635 upper=1.9635 effort=0 velocity=0.2 -> lower=0 upper=1.9635 effort=0 velocity=0.2
- joint r_sho_roll: limit lower=-1.9635 upper=0 effort=87 velocity=1.5 -> lower=-1.9635 upper=1.9635 effort=87 velocity=1.5
