Commit message: add diablocustom4 (dumbell)

File: assets/urdf/dumbbell.urdf (robot description, URDF)
Before this commit: robot dumbbell, 3 links, 2 joints
Links:
- added link handle_target; visual sphere radius=0.005
- link handle: geometry collision cylinder length=0.10 radius=0.01; visual cylinder length=0.10 radius=0.01
Joints:
- added joint joint_target: type fixed, parent handle, child handle_target, origin xyz=0 0 0 rpy=0 0 0

Commit message: Adding dumbbell configs.

File: assets/urdf/dumbbell.urdf (robot description, URDF)
Before this commit: robot dumbbell, 4 links, 3 joints
Links:
- link handle: mass 0.5 -> 0.02; geometry collision cylinder length=0.08 radius=0.006; visual cylinder length=0.08 radius=0.006
- link handle_target: geometry visual sphere radius=0.003
- link left_weight: mass 1.0 -> 0.04; geometry collision cylinder length=0.024 radius=0.024; visual cylinder length=0.024 radius=0.024
- link right_weight: mass 1.0 -> 0.04; geometry collision cylinder length=0.024 radius=0.024; visual cylinder length=0.024 radius=0.024
