Commit message: change mug path

File: assets/urdf/ycb/025_mug/025_mug.urdf (robot description, URDF)
Before this commit: robot mug, 1 links, 0 joints
Links:
- added link handle_target; visual sphere radius=0.005
Joints:
- added joint mug_to_handle: type fixed, parent mug, child handle_target, origin xyz=0.065 0.0 0.005 rpy=0 0 0
